File: Eagle/FizziLagTester.brd (EAGLE design)
At the start: 100.3 x 80 mm, 36 parts, among them J2 AVR_SPI_PRG_6PTH, Y2 16MHz

Commit message: I think revision 1.1 should be functional...
Parts:
- removed JGC3, JGC4: (no value), SparkFun-Connectors:1X02
- removed R19: PHOTOCELLPTH, SparkFun-Sensors:PHOTOCELL
- removed R22: 10k, SparkFun-Passives:0603-RES
Connections:
- removed net VOLS2: LSENSOR2.2, R18.1
- removed net VOLS3: R19.1, R22.1
- net 5V: no longer JGC3.1, JGC4.1, R19.2
- net GND: no longer R22.2
- net VOLS: now also LSENSOR2.2, R18.1; no longer JGC3.2, JGC4.2
Routing:
- net VOLS2: track 83.5 -> 0.00 mm, vias 2 -> 0
- net VOLS3: track 54.2 -> 0.00 mm, vias 1 -> 0
- net 5V: track 223.7 -> 198.6 mm, vias 6 -> 4
- net VOLS: track 84.4 -> 64.2 mm, vias 3 -> 2
- net N$18: track 0.00 -> 2.57 mm
- net AUDIO: track 108.3 -> 110.2 mm
Other:
- board text added: "Revision 1.1"
