File: Eagle/FizziLagTester.sch (EAGLE design)
At the start: 36 parts, among them J2 AVR_SPI_PRG_6PTH, Y2 16MHz

Commit message: I think revision 1.1 should be functional...
Parts:
- removed JGC3, JGC4: (no value), SparkFun-Connectors:M02PTH
- removed R19: PHOTOCELLPTH, SparkFun-Sensors:PHOTOCELLPTH
- removed R22: 10k, SparkFun-Passives:RESISTOR0603-RES
Connections:
- removed net VOLS2: LSENSOR2.-, R18.1
- removed net VOLS3: R19.P$1, R22.1
- net 5V: no longer JGC3.1, JGC4.1, R19.P$2
- net GND: no longer R22.2
- net VOLS: now also LSENSOR2.-, R18.1; no longer JGC3.2, JGC4.2
Changed lines of the file:
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@@
 <part name="R18" library="SparkFun-Passives" deviceset="RESISTOR" device="0603-RES" value="5k"/>
 <part name="U$4" library="SparkFun" deviceset="5V" device=""/>
-<part name="R19" library="SparkFun-Sensors" deviceset="PHOTOCELL" device="PTH"/>
-<part name="U$6" library="SparkFun" deviceset="5V" device=""/>
-<part name="GND14" library="SparkFun" deviceset="GND" device=""/>
-<part name="R22" library="SparkFun-Passives" deviceset="RESISTOR" device="0603-RES" value="10k"/>
-<part name="JGC3" library="SparkFun-Connectors" deviceset="M02" device="PTH"/>
-<part name="JGC4" library="SparkFun-Connectors" deviceset="M02" device="PTH"/>
-<part name="U$12" library="SparkFun" deviceset="5V" device=""/>
-<part name="U$13" library="SparkFun" deviceset="5V" device=""/>
 <part name="C1" library="SparkFun-Capacitors" deviceset="CAP_POL" device="PTH1" value="47u"/>
 <part name="C2" library="SparkFun-Capacitors" deviceset="CAP_POL" device="PTH1" value="47u"/>
@@
 <instance part="R18" gate="G$1" x="-20.32" y="121.92" rot="R270"/>
 <instance part="U$4" gate="G$1" x="-20.32" y="157.48"/>
-<instance part="R19" gate="G$1" x="15.24" y="144.78" rot="R90"/>
-<instance part="U$6" gate="G$1" x="15.24" y="157.48"/>
-<instance part="GND14" gate="1" x="15.24" y="106.68"/>
-<instance part="R22" gate="G$1" x="15.24" y="121.92" rot="R270"/>
-<instance part="JGC3" gate="G$1" x="114.3" y="71.12" rot="R180"/>
-<instance part="JGC4" gate="G$1" x="114.3" y="48.26" rot="R180"/>
-<instance part="U$12" gate="G$1" x="104.14" y="73.66"/>
-<instance part="U$13" gate="G$1" x="104.14" y="50.8"/>
 <instance part="C1" gate="G$1" x="12.7" y="-5.08"/>
 <instance part="C2" gate="G$1" x="58.42" y="-2.54"/>
@@
 <wire x1="-20.32" y1="109.22" x2="-20.32" y2="116.84" width="0.1524" layer="91"/>
 </segment>
-<segment>
-<pinref part="R22" gate="G$1" pin="2"/>
-<pinref part="GND14" gate="1" pin="GND"/>
-<wire x1="15.24" y1="116.84" x2="15.24" y2="109.22" width="0.1524" layer="91"/>
-</segment>
 </net>
 <net name="VOLS" class="0">
@@
 </segment>
 <segment>
-<pinref part="JGC4" gate="G$1" pin="2"/>
-<wire x1="106.68" y1="45.72" x2="101.6" y2="45.72" width="0.1524" layer="91"/>
-<wire x1="101.6" y1="45.72" x2="101.6" y2="58.42" width="0.1524" layer="91"/>
-<pinref part="JGC3" gate="G$1" pin="2"/>
-<wire x1="106.68" y1="68.58" x2="101.6" y2="68.58" width="0.1524" layer="91"/>
-<wire x1="101.6" y1="68.58" x2="101.6" y2="58.42" width="0.1524" layer="91"/>
-<wire x1="88.9" y1="58.42" x2="101.6" y2="58.42" width="0.1524" layer="91"/>
-<junction x="101.6" y="58.42"/>
-<label x="88.9" y="58.42" size="1.778" layer="95"/>
+<pinref part="R18" gate="G$1" pin="1"/>
+<pinref part="LSENSOR2" gate="G$1" pin="-"/>
+<wire x1="-20.32" y1="127" x2="-20.32" y2="134.62" width="0.1524" layer="91"/>
+<wire x1="-20.32" y1="134.62" x2="-20.32" y2="142.24" width="0.1524" layer="91"/>
+<wire x1="-20.32" y1="134.62" x2="-38.1" y2="134.62" width="0.1524" layer="91"/>
+<label x="-38.1" y="134.62" size="1.778" layer="95"/>
+<junction x="-20.32" y="134.62"/>
 </segment>
 </net>
@@
 <wire x1="-20.32" y1="149.86" x2="-20.32" y2="157.48" width="0.1524" layer="91"/>
 </segment>
-<segment>
-<pinref part="U$6" gate="G$1" pin="5V"/>
-<pinref part="R19" gate="G$1" pin="P$2"/>
-<wire x1="15.24" y1="157.48" x2="15.24" y2="152.4" width="0.1524" layer="91"/>
-</segment>
-<segment>
-<pinref part="JGC3" gate="G$1" pin="1"/>
-<wire x1="106.68" y1="71.12" x2="104.14" y2="71.12" width="0.1524" layer="91"/>
-<wire x1="104.14" y1="71.12" x2="104.14" y2="73.66" width="0.1524" layer="91"/>
-<pinref part="U$12" gate="G$1" pin="5V"/>
-</segment>
-<segment>
-<pinref part="JGC4" gate="G$1" pin="1"/>
-<wire x1="106.68" y1="48.26" x2="104.14" y2="48.26" width="0.1524" layer="91"/>
-<wire x1="104.14" y1="48.26" x2="104.14" y2="50.8" width="0.1524" layer="91"/>
-<pinref part="U$13" gate="G$1" pin="5V"/>
-</segment>
 </net>
 <net name="N$3" class="0">
@@
 </segment>
 </net>
-<net name="VOLS2" class="0">
-<segment>
-<pinref part="R18" gate="G$1" pin="1"/>
-<pinref part="LSENSOR2" gate="G$1" pin="-"/>
-<wire x1="-20.32" y1="127" x2="-20.32" y2="134.62" width="0.1524" layer="91"/>
-<wire x1="-20.32" y1="134.62" x2="-20.32" y2="142.24" width="0.1524" layer="91"/>
-<wire x1="-20.32" y1="134.62" x2="-38.1" y2="134.62" width="0.1524" layer="91"/>
-<label x="-38.1" y="134.62" size="1.778" layer="95"/>
-<junction x="-20.32" y="134.62"/>
-</segment>
-</net>
-<net name="VOLS3" class="0">
-<segment>
-<wire x1="15.24" y1="134.62" x2="0" y2="134.62" width="0.1524" layer="91"/>
-<label x="0" y="134.62" size="1.778" layer="95"/>
-<pinref part="R19" gate="G$1" pin="P$1"/>
-<pinref part="R22" gate="G$1" pin="1"/>
-<wire x1="15.24" y1="137.16" x2="15.24" y2="134.62" width="0.1524" layer="91"/>
-<junction x="15.24" y="134.62"/>
-<wire x1="15.24" y1="134.62" x2="15.24" y2="127" width="0.1524" layer="91"/>
-</segment>
-</net>
